File: Minutnix I ver/MainBoard.sch (EAGLE design)
At the start: 32 parts, among them IC1 MEGA8-AI, Q1 32.768kHz

Commit message: Minor board changes
Parts:
- added Q2: (no value), semicon-smd-ipc:NPN-TRANSISTOR_SOT23
- added R30: 4.7k, rcl:R-EU_01005
- added SG1: F/CM12P, buzzer:F/CM12P
Connections:
- new net N$43: IC1.PB2(SS/OC1B), R30.2
- new net N$51: Q2.B, R30.1
- new net N$52: Q2.C, SG1.2
- net GND: now also Q2.E
- net VCC: now also SG1.1
